Commit message: Update robot dimensions in URDF for improved accuracy

File: susumu_diffbot/description/urdf/diffbot.urdf.xacro (robot description, xacro)
@@ -4,9 +4,9 @@
   <xacro:arg name="prefix" default="" />
   <xacro:arg name="use_mock_hardware" default="false" />
-  <xacro:include filename="$(find odrive_botwheel_explorer)/urdf/diffbot_description.urdf.xacro" />
+  <xacro:include filename="$(find susumu_diffbot)/description/urdf/diffbot_description.urdf.xacro" />
   <!-- Import Rviz colors -->
-  <!--<xacro:include filename="$(find odrive_botwheel_explorer)/urdf/diffbot.materials.xacro" />-->
+  <!--<xacro:include filename="$(find susumu_diffbot)/description/urdf/diffbot.materials.xacro" />-->
   <!-- Import diffbot ros2_control description -->
-  <xacro:include filename="$(find odrive_botwheel_explorer)/urdf/diffbot.ros2_control.xacro" />
+  <xacro:include filename="$(find susumu_diffbot)/description/urdf/diffbot.ros2_control.xacro" />
   <xacro:diffbot prefix="$(arg prefix)" />
   <xacro:diffbot_ros2_control

File: susumu_diffbot/description/urdf/diffbot_description.urdf.xacro (robot description, xacro)
@@ -5,7 +5,7 @@
   <xacro:property name="PI" value="3.1415926535897931"/>
   <xacro:property name="base_mass" value="0.3" /> <!-- arbitrary value for base mass -->
-  <xacro:property name="base_width" value="0.1" />
-  <xacro:property name="base_length" value="0.1" />
-  <xacro:property name="base_height" value="0.05" />
+  <xacro:property name="base_width" value="0.21" />
+  <xacro:property name="base_length" value="0.35" />
+  <xacro:property name="base_height" value="0.31" />
   <xacro:property name="wheel_mass" value="0.3" /> <!-- arbitrary value for wheel mass -->
   <xacro:property name="wheel_len" value="0.020" />
