Commit message: Fix wheel separation and offset to match actual hardware dimensions
wheel_separation: 0.134 → 0.255
wheel_offset_y: 0.08 → 0.1275

Co-Authored-By: Claude Sonnet 4.6 <noreply@anthropic.com>

File: susumu_diffbot/urdf/diffbot_description.urdf.xacro (robot description, xacro)
@@ -11,5 +11,5 @@
     <xacro:property name="wheel_mass" value="0.05"/>
     <xacro:property name="wheel_offset_x" value="-0.18"/>
-    <xacro:property name="wheel_offset_y" value="0.08"/>
+    <xacro:property name="wheel_offset_y" value="0.1275"/>
     <xacro:property name="wheel_offset_z" value="0.07"/>
     <xacro:property name="caster_wheel_radius" value="0.01"/>

Commit message: Fix wheel_offset_x to 0.0 to center wheels on base_link
Co-Authored-By: Claude Sonnet 4.6 <noreply@anthropic.com>

File: susumu_diffbot/urdf/diffbot_description.urdf.xacro (robot description, xacro)
@@ -10,5 +10,5 @@
     <xacro:property name="wheel_thickness" value="0.043"/>
     <xacro:property name="wheel_mass" value="0.05"/>
-    <xacro:property name="wheel_offset_x" value="-0.18"/>
+    <xacro:property name="wheel_offset_x" value="0.0"/>
     <xacro:property name="wheel_offset_y" value="0.1275"/>
     <xacro:property name="wheel_offset_z" value="0.07"/>
