Commit message: Add Gazebo Classic simulation stack alongside real-robot launches
Brings up the full robo_indoor + nav2 pipeline on Gazebo without
any physical hardware (mic / speaker / LiDAR / camera / motors / GNSS).

- URDF: add use_gazebo arg to switch between ODrive and gazebo_ros2_control,
  add depth camera (D435i-equivalent), drop /diffbot namespace from IMU
- New launches: sim_robot, robo_indoor_sim, nav2_sim, slam_toolbox_sim,
  collision_monitor_sim, dummy_audio, audio_option_sim
- New node: dummy_speak_action_server (offline /speak action)
- Raise controller_manager update_rate to 100 Hz for Gazebo sim
- Register sim entries in the GUI menu and update README / AGENTS docs

Co-Authored-By: Claude Opus 4.7 <noreply@anthropic.com>

File: susumu_diffbot/urdf/diffbot.ros2_control.xacro (robot description, xacro)
@@ -1,25 +1,45 @@
 <?xml version="1.0"?>
 <robot xmlns:xacro="http://www.ros.org/wiki/xacro">
-  <xacro:macro name="diffbot_ros2_control" params="name prefix use_mock_hardware">
+  <xacro:macro name="diffbot_ros2_control" params="name prefix use_mock_hardware use_gazebo:=false">
     <ros2_control name="${name}" type="system">
-      <xacro:unless value="${use_mock_hardware}">
+      <xacro:if value="${use_gazebo}">
         <hardware>
-          <plugin>odrive_ros2_control_plugin/ODriveHardwareInterface</plugin>
-          <param name="can">can0</param>
-        </hardware>
-      </xacro:unless>
-      <xacro:if value="${use_mock_hardware}">
-        <hardware>
-          <plugin>mock_components/GenericSystem</plugin>
-          <param name="calculate_dynamics">true</param>
+          <plugin>gazebo_ros2_control/GazeboSystem</plugin>
         </hardware>
       </xacro:if>
+      <xacro:unless value="${use_gazebo}">
+        <xacro:unless value="${use_mock_hardware}">
+          <hardware>
+            <plugin>odrive_ros2_control_plugin/ODriveHardwareInterface</plugin>
+            <param name="can">can0</param>
+          </hardware>
+        </xacro:unless>
+        <xacro:if value="${use_mock_hardware}">
+          <hardware>
+            <plugin>mock_components/GenericSystem</plugin>
+            <param name="calculate_dynamics">true</param>
+          </hardware>
+        </xacro:if>
+      </xacro:unless>
       <joint name="${prefix}left_wheel_joint">
         <param name="node_id">0</param>
+        <command_interface name="velocity"/>
+        <state_interface name="velocity"/>
+        <state_interface name="position"/>
       </joint>
       <joint name="${prefix}right_wheel_joint">
         <param name="node_id">1</param>
+        <command_interface name="velocity"/>
+        <state_interface name="velocity"/>
+        <state_interface name="position"/>
       </joint>
     </ros2_control>
+    <xacro:if value="${use_gazebo}">
+      <gazebo>
+        <plugin name="gazebo_ros2_control" filename="libgazebo_ros2_control.so">
+          <parameters>$(find susumu_robo)/susumu_diffbot/config/diffbot_controllers.yaml</parameters>
+        </plugin>
+      </gazebo>
+    </xacro:if>
   </xacro:macro>
 </robot>

File: susumu_diffbot/urdf/diffbot.urdf.xacro (robot description, xacro)
@@ -5,13 +5,17 @@
   <xacro:arg name="use_ros2_control" default="true"/>
   <xacro:arg name="use_mock_hardware" default="false"/>
+  <xacro:arg name="use_gazebo" default="false"/>
   <xacro:include filename="$(find susumu_robo)/susumu_diffbot/urdf/inertial_macros.xacro"/>
   <xacro:include filename="$(find susumu_robo)/susumu_diffbot/urdf/diffbot_description.urdf.xacro"/>
   <xacro:include filename="$(find susumu_robo)/susumu_diffbot/urdf/imu.xacro"/>
   <xacro:include filename="$(find susumu_robo)/susumu_diffbot/urdf/lidar.xacro"/>
+  <xacro:include filename="$(find susumu_robo)/susumu_diffbot/urdf/camera.xacro"/>
   <xacro:diffbot prefix="$(arg prefix)" />
   <xacro:if value="$(arg use_ros2_control)">
     <xacro:include filename="$(find susumu_robo)/susumu_diffbot/urdf/diffbot.ros2_control.xacro"/>
     <xacro:diffbot_ros2_control
-      name="DiffBot" prefix="$(arg prefix)" use_mock_hardware="$(arg use_mock_hardware)"/>
+      name="DiffBot" prefix="$(arg prefix)"
+      use_mock_hardware="$(arg use_mock_hardware)"
+      use_gazebo="$(arg use_gazebo)"/>
   </xacro:if>
 </robot>

File: susumu_diffbot/urdf/imu.xacro (robot description, xacro)
@@ -25,8 +25,8 @@
         <plugin filename="libgazebo_ros_imu_sensor.so" name="imu_plugin">
             <ros>
-                <namespace>/diffbot</namespace>
-                <remapping>~/out:=imu</remapping>
+                <remapping>~/out:=imu/data</remapping>
             </ros>
             <initial_orientation_as_reference>false</initial_orientation_as_reference>
+            <frame_name>imu_link</frame_name>
             </plugin>
             <always_on>true</always_on>
